File: electronics/stm32-e407-shield/schematic.sch (EAGLE design)
At the start: 36 parts, among them IC1 MAX3468CPA, IC2 LM340H-12, IC3 LM340H-12

Commit message: Alterações no Shield para ARM e biblioteca padrão.
O conversor lógico foi modelado no Eagle e adicionado à recem criada
biblioteca provant_custom.lbr. Ele foi então usado para substituir
o coversor lógico hard-core que havia sido previamente projetado.

Planos para remover o IMU_SLC - ele agora influencia a tensão do
barramento do ESC, o que não é desejado.

	new file:   .gitignore
	new file:   lib/.gitignore
	new file:   lib/provant_custom.lbr
	modified:   stm32-e407-shield/schematic.brd
	modified:   stm32-e407-shield/schematic.sch
Parts:
- removed JP1, JP2: 0, adafruit:R-US_M1406
- removed Q1, Q2, Q3, Q4, Q5: (no value), adafruit:MOSFET-NREFLOW
- removed R3, R5: 4k7, adafruit:R-US_M1406
- added T1: 2N3565, transistor:2N3565
- added U$1: JYMCU_LOGIC_LEVEL_CONVERTER, provant_custom:JYMCU_LOGIC_LEVEL_CONVERTER
Connections:
- removed net N$2: ESC.3, ESC.4, Q1.D
- removed net N$4: ESC.5, ESC.6, Q2.D
- removed net N$5: IMU.3, JP2.2, Q4.D, R3.2
- new net N$12: ESC.5, ESC.6, IMU.3, U$1.B_L
- net 3.3V: no longer Q1.G, Q2.G, Q3.G, Q4.G
- net 5V: now also U$1.5V
- net GND: now also T1.E, U$1.GND1, U$1.GND2; no longer Q5.S
- net N$1: now also U$1.3V3, VIMU_SLC.2; no longer IMU.4, JP1.2, Q3.D, R5.2
- net N$6: now also T1.B; no longer Q5.G
- net N$7: now also ESC.3, ESC.4, U$1.A_L; no longer JP1.1, JP2.1, R3.1, R5.1, VIMU_SLC.2
- net PB8_I2C1_SCL: now also U$1.A_H; no longer Q2.S, Q3.S
- net PB9_I2C1_SDA: now also U$1.B_H; no longer Q1.S, Q4.S
- net PC7_USART6_RX: now also T1.C; no longer Q5.D
Other:
- note removed: "JP1 e JP2 curto circuitam os Pull-Ups da I2C caso necessário."
- moved on the sheet: ESC, IMU, VIMU_SLC

Commit message: Versão dual layer pra fabricação manual.
Parts:
- R1, R4: device adafruit:R-US_M1406 -> adafruit:R-US_0309/V
- R2, R7: device adafruit:R-US_M1406 -> adafruit:R-US_0204/7
Changed lines of the file:
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@@
 <part name="GND15" library="SparkFun-Aesthetics" deviceset="GND" device=""/>
 <part name="GND16" library="SparkFun-Aesthetics" deviceset="GND" device=""/>
-<part name="R1" library="adafruit" deviceset="R-US_" device="M1406" value="4k7"/>
-<part name="R2" library="adafruit" deviceset="R-US_" device="M1406" value="4k7"/>
-<part name="R4" library="adafruit" deviceset="R-US_" device="M1406" value="4k7"/>
-<part name="R7" library="adafruit" deviceset="R-US_" device="M1406" value="4k7"/>
+<part name="R1" library="adafruit" deviceset="R-US_" device="0309/V" value="4k7"/>
+<part name="R2" library="adafruit" deviceset="R-US_" device="0204/7" value="4k7"/>
+<part name="R4" library="adafruit" deviceset="R-US_" device="0309/V" value="4k7"/>
+<part name="R7" library="adafruit" deviceset="R-US_" device="0204/7" value="4k7"/>
 <part name="LED1" library="adafruit" deviceset="LED" device="3MM"/>
 <part name="LED2" library="adafruit" deviceset="LED" device="3MM"/>

Commit message: Pequenas correções depois da primeira tentativa de fabricação.
Connections:
- net N$1: now also IMU.4
Changed lines of the file:
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@@
 <grid distance="0.1" unitdist="inch" unit="inch" style="lines" multiple="1" display="no" altdistance="0.01" altunitdist="inch" altunit="inch"/>
 <layers>
-<layer number="1" name="Top" color="4" fill="1" visible="yes" active="no"/>
-<layer number="16" name="Bottom" color="1" fill="1" visible="yes" active="no"/>
-<layer number="17" name="Pads" color="2" fill="1" visible="yes" active="no"/>
-<layer number="18" name="Vias" color="2" fill="1" visible="yes" active="no"/>
-<layer number="19" name="Unrouted" color="6" fill="1" visible="yes" active="no"/>
-<layer number="20" name="Dimension" color="15" fill="1" visible="yes" active="no"/>
-<layer number="21" name="tPlace" color="7" fill="1" visible="yes" active="no"/>
-<layer number="22" name="bPlace" color="7" fill="1" visible="yes" active="no"/>
-<layer number="23" name="tOrigins" color="15" fill="1" visible="yes" active="no"/>
-<layer number="24" name="bOrigins" color="15" fill="1" visible="yes" active="no"/>
-<layer number="25" name="tNames" color="7" fill="1" visible="yes" active="no"/>
-<layer number="26" name="bNames" color="7" fill="1" visible="yes" active="no"/>
-<layer number="27" name="tValues" color="7" fill="1" visible="yes" active="no"/>
-<layer number="28" name="bValues" color="7" fill="1" visible="yes" active="no"/>
+<layer number="1" name="Top" color="4" fill="1" visible="no" active="no"/>
+<layer number="16" name="Bottom" color="1" fill="1" visible="no" active="no"/>
+<layer number="17" name="Pads" color="2" fill="1" visible="no" active="no"/>
+<layer number="18" name="Vias" color="2" fill="1" visible="no" active="no"/>
+<layer number="19" name="Unrouted" color="6" fill="1" visible="no" active="no"/>
+<layer number="20" name="Dimension" color="15" fill="1" visible="no" active="no"/>
+<layer number="21" name="tPlace" color="7" fill="1" visible="no" active="no"/>
+<layer number="22" name="bPlace" color="7" fill="1" visible="no" active="no"/>
+<layer number="23" name="tOrigins" color="15" fill="1" visible="no" active="no"/>
+<layer number="24" name="bOrigins" color="15" fill="1" visible="no" active="no"/>
+<layer number="25" name="tNames" color="7" fill="1" visible="no" active="no"/>
+<layer number="26" name="bNames" color="7" fill="1" visible="no" active="no"/>
+<layer number="27" name="tValues" color="7" fill="1" visible="no" active="no"/>
+<layer number="28" name="bValues" color="7" fill="1" visible="no" active="no"/>
 <layer number="29" name="tStop" color="7" fill="3" visible="no" active="no"/>
 <layer number="30" name="bStop" color="7" fill="6" visible="no" active="no"/>
@@
 <layer number="35" name="tGlue" color="7" fill="4" visible="no" active="no"/>
 <layer number="36" name="bGlue" color="7" fill="5" visible="no" active="no"/>
-<layer number="37" name="tTest" color="7" fill="1" visible="yes" active="no"/>
-<layer number="38" name="bTest" color="7" fill="1" visible="yes" active="no"/>
+<layer number="37" name="tTest" color="7" fill="1" visible="no" active="no"/>
+<layer number="38" name="bTest" color="7" fill="1" visible="no" active="no"/>
 <layer number="39" name="tKeepout" color="4" fill="11" visible="no" active="no"/>
 <layer number="40" name="bKeepout" color="1" fill="11" visible="no" active="no"/>
@@
 <layer number="44" name="Drills" color="7" fill="1" visible="no" active="no"/>
 <layer number="45" name="Holes" color="7" fill="1" visible="no" active="no"/>
-<layer number="46" name="Milling" color="3" fill="1" visible="yes" active="no"/>
-<layer number="47" name="Measures" color="7" fill="1" visible="yes" active="no"/>
-<layer number="48" name="Document" color="7" fill="1" visible="yes" active="no"/>
-<layer number="49" name="Reference" color="7" fill="1" visible="yes" active="no"/>
-<layer number="50" name="dxf" color="7" fill="1" visible="yes" active="no"/>
-<layer number="51" name="tDocu" color="7" fill="1" visible="yes" active="no"/>
-<layer number="52" name="bDocu" color="7" fill="1" visible="yes" active="no"/>
-<layer number="53" name="tGND_GNDA" color="7" fill="9" visible="yes" active="no"/>
-<layer number="54" name="bGND_GNDA" color="1" fill="9" visible="yes" active="no"/>
-<layer number="56" name="wert" color="7" fill="1" visible="yes" active="no"/>
-<layer number="57" name="tCAD" color="7" fill="1" visible="yes" active="no"/>
+<layer number="46" name="Milling" color="3" fill="1" visible="no" active="no"/>
+<layer number="47" name="Measures" color="7" fill="1" visible="no" active="no"/>
+<layer number="48" name="Document" color="7" fill="1" visible="no" active="no"/>
+<layer number="49" name="Reference" color="7" fill="1" visible="no" active="no"/>
+<layer number="50" name="dxf" color="7" fill="1" visible="no" active="no"/>
+<layer number="51" name="tDocu" color="7" fill="1" visible="no" active="no"/>
+<layer number="52" name="bDocu" color="7" fill="1" visible="no" active="no"/>
+<layer number="53" name="tGND_GNDA" color="7" fill="9" visible="no" active="no"/>
+<layer number="54" name="bGND_GNDA" color="1" fill="9" visible="no" active="no"/>
+<layer number="56" name="wert" color="7" fill="1" visible="no" active="no"/>
+<layer number="57" name="tCAD" color="7" fill="1" visible="no" active="no"/>
 <layer number="91" name="Nets" color="2" fill="1" visible="yes" active="yes"/>
 <layer number="92" name="Busses" color="1" fill="1" visible="yes" active="yes"/>
@@
 <pinref part="U$1" gate="G$1" pin="3V3"/>
 <wire x1="20.32" y1="142.24" x2="22.86" y2="142.24" width="0.1524" layer="91"/>
-</segment>
-</net>
+<wire x1="20.32" y1="162.56" x2="20.32" y2="172.72" width="0.1524" layer="91"/>
+<pinref part="IMU" gate="G$1" pin="4"/>
+<wire x1="20.32" y1="172.72" x2="-10.16" y2="172.72" width="0.1524" layer="91"/>
+<junction x="20.32" y="162.56"/>
+</segment>
+</net>
