File: electronics/stm32f4discovery-shield/schematic.sch (EAGLE design)
At the start: 40 parts, among them IC1 MAX3468CPA, IC3 LM340H-12, IC4 LM340H-12, J1 POWER_JACKSLT, Q1 BC548

Commit message: Adicionadas algumas correcoes.
Parts:
- renumbered U$2 to LVL
Other:
- note added: "Layers (p/ silk e top/bottom) - 1, 16 17, 18, 20, 21, 22, 25, 26, 48, 49, 51, 52"
