File: electronics/stm32f4discovery-shield/schematic.sch (EAGLE design)
At the start: 40 parts, among them IC1 MAX3468CPA, IC3 LM340H-12, IC4 LM340H-12, J1 POWER_JACKSLT, Q1 BC548

Commit message: Iniciando revisao da shield Discovery.
Parts:
- renumbered LVL to U$2
Changed lines of the file:
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@@
 <?xml version="1.0" encoding="utf-8"?>
 <!DOCTYPE eagle SYSTEM "eagle.dtd">
-<eagle version="6.5.0">
+<eagle version="6.4">
 <drawing>
 <settings>
@@
 <part name="GND9" library="SparkFun-Aesthetics" deviceset="GND" device=""/>
 <part name="GND10" library="SparkFun-Aesthetics" deviceset="GND" device=""/>
-<part name="LVL" library="provant_custom" deviceset="JYMCU_LOGIC_LEVEL_CONVERTER" device=""/>
+<part name="U$2" library="provant_custom" deviceset="JYMCU_LOGIC_LEVEL_CONVERTER" device=""/>
 <part name="I2C1_ESC" library="con-tycoelectronics" deviceset="RJ11" device="" technology="-2L-B"/>
 <part name="I2C3_IMU" library="con-tycoelectronics" deviceset="RJ11" device="" technology="-2L-B"/>
@@
 <instance part="GND9" gate="1" x="22.86" y="63.5" rot="R270"/>
 <instance part="GND10" gate="1" x="22.86" y="40.64" rot="R270"/>
-<instance part="LVL" gate="G$1" x="63.5" y="149.86"/>
+<instance part="U$2" gate="G$1" x="63.5" y="149.86"/>
 <instance part="I2C1_ESC" gate="G$1" x="132.08" y="160.02"/>
 <instance part="I2C3_IMU" gate="G$1" x="132.08" y="134.62"/>
@@
 </segment>
 <segment>
-<pinref part="LVL" gate="G$1" pin="GND2"/>
+<pinref part="U$2" gate="G$1" pin="GND2"/>
 <pinref part="GND31" gate="1" pin="GND"/>
 </segment>
 <segment>
-<pinref part="LVL" gate="G$1" pin="GND1"/>
+<pinref part="U$2" gate="G$1" pin="GND1"/>
 <pinref part="GND32" gate="1" pin="GND"/>
 </segment>
@@
 </segment>
 <segment>
-<pinref part="LVL" gate="G$1" pin="5V"/>
+<pinref part="U$2" gate="G$1" pin="5V"/>
 <pinref part="SUPPLY32" gate="G$1" pin="5V"/>
 <wire x1="78.74" y1="157.48" x2="78.74" y2="154.94" width="0.1524" layer="91"/>
@@
 </segment>
 <segment>
-<pinref part="LVL" gate="G$1" pin="3V3"/>
+<pinref part="U$2" gate="G$1" pin="3V3"/>
 <pinref part="SUPPLY31" gate="G$1" pin="3.3V"/>
 <wire x1="48.26" y1="157.48" x2="48.26" y2="154.94" width="0.1524" layer="91"/>
@@
 <pinref part="JP1" gate="1" pin="5"/>
 <wire x1="45.72" y1="132.08" x2="45.72" y2="142.24" width="0.1524" layer="91"/>
-<pinref part="LVL" gate="G$1" pin="D_L"/>
+<pinref part="U$2" gate="G$1" pin="D_L"/>
 <wire x1="45.72" y1="142.24" x2="48.26" y2="142.24" width="0.1524" layer="91"/>
 </segment>
@@
 <net name="N$2" class="0">
 <segment>
-<pinref part="LVL" gate="G$1" pin="C_L"/>
+<pinref part="U$2" gate="G$1" pin="C_L"/>
 <wire x1="48.26" y1="144.78" x2="43.18" y2="144.78" width="0.1524" layer="91"/>
 <wire x1="43.18" y1="144.78" x2="43.18" y2="114.3" width="0.1524" layer="91"/>
@@
 <wire x1="81.28" y1="134.62" x2="50.8" y2="134.62" width="0.1524" layer="91"/>
 <wire x1="50.8" y1="134.62" x2="50.8" y2="132.08" width="0.1524" layer="91"/>
-<pinref part="LVL" gate="G$1" pin="D_H"/>
+<pinref part="U$2" gate="G$1" pin="D_H"/>
 <wire x1="78.74" y1="142.24" x2="81.28" y2="142.24" width="0.1524" layer="91"/>
 <wire x1="81.28" y1="142.24" x2="81.28" y2="134.62" width="0.1524" layer="91"/>
@@
 <wire x1="53.34" y1="114.3" x2="50.8" y2="114.3" width="0.1524" layer="91"/>
 <wire x1="50.8" y1="114.3" x2="50.8" y2="116.84" width="0.1524" layer="91"/>
-<pinref part="LVL" gate="G$1" pin="C_H"/>
+<pinref part="U$2" gate="G$1" pin="C_H"/>
 <wire x1="78.74" y1="144.78" x2="83.82" y2="144.78" width="0.1524" layer="91"/>
 <wire x1="83.82" y1="144.78" x2="83.82" y2="132.08" width="0.1524" layer="91"/>
@@
 <wire x1="114.3" y1="160.02" x2="83.82" y2="160.02" width="0.1524" layer="91"/>
 <wire x1="83.82" y1="160.02" x2="83.82" y2="149.86" width="0.1524" layer="91"/>
-<pinref part="LVL" gate="G$1" pin="A_H"/>
+<pinref part="U$2" gate="G$1" pin="A_H"/>
 <wire x1="83.82" y1="149.86" x2="78.74" y2="149.86" width="0.1524" layer="91"/>
 <wire x1="111.76" y1="170.18" x2="114.3" y2="170.18" width="0.1524" layer="91"/>
@@
 <wire x1="111.76" y1="157.48" x2="86.36" y2="157.48" width="0.1524" layer="91"/>
 <wire x1="86.36" y1="157.48" x2="86.36" y2="147.32" width="0.1524" layer="91"/>
-<pinref part="LVL" gate="G$1" pin="B_H"/>
+<pinref part="U$2" gate="G$1" pin="B_H"/>
 <wire x1="86.36" y1="147.32" x2="78.74" y2="147.32" width="0.1524" layer="91"/>
 <wire x1="111.76" y1="167.64" x2="111.76" y2="157.48" width="0.1524" layer="91"/>
@@
 <net name="PB9/I2C1_SDA" class="0">
 <segment>
-<pinref part="LVL" gate="G$1" pin="A_L"/>
+<pinref part="U$2" gate="G$1" pin="A_L"/>
 <wire x1="48.26" y1="149.86" x2="10.16" y2="149.86" width="0.1524" layer="91"/>
 <label x="10.16" y="149.86" size="1.778" layer="95"/>
@@
 <net name="PB8/I2C1_SCL" class="0">
 <segment>
-<pinref part="LVL" gate="G$1" pin="B_L"/>
+<pinref part="U$2" gate="G$1" pin="B_L"/>
 <wire x1="48.26" y1="147.32" x2="10.16" y2="147.32" width="0.1524" layer="91"/>
 <label x="10.16" y="147.32" size="1.778" layer="95"/>

Commit message: Alterado o layout da placa, removidas algumas frescuras.
Parts:
- added R11: (no value), adafruit:R-US_M1406
- R1, R3: device adafruit:R-US_M1206 -> adafruit:R-US_M1406
- R10, R9: device adafruit:R-US_0204/7 -> adafruit:R-US_0204/2V
- R2: device rcl:R-EU_0204/5 -> rcl:R-EU_0204/7
- renumbered JP1 to SV4
Connections:
- new net N$9: I2C3_IMU.6, R11.2
- new net PD3: IC1.DE, IC1.RE/, U$1.PD3
- net 3.3V: now also R11.1; no longer I2C3_IMU.1
- net GND: no longer I2C3_IMU.6
- net N$1: now also SV4.6; no longer SV4.5
- net N$2: now also SV4.5; no longer SV4.6
- net PA8/I2C3_SCL: now also SV4.3; no longer SV4.4
- net PB0/PWM: now also LED2.C; no longer LED1.C
- net PB1/PWM: now also LED1.C; no longer LED2.C
- net PC9/I2C3_SDA: now also SV4.4; no longer SV4.3
- net PE2: no longer IC1.DE, IC1.RE/
- net SCL2: now also SV4.1; no longer SV4.2
- net SDA2: now also SV4.2; no longer SV4.1

Commit message: Adicionado o jack para sensores analógicos. LEDs trocados para LEDs de 3mm. Verificaçao de routing do GND feita - aparentemente, sem problemas.
Parts:
- added AN1: RJ11-2L-B, con-tycoelectronics:RJ11-2L-B
- added JP1: (no value), jumper:JP2E
- C2: device SparkFun-Capacitors:0.1UF-50V-20%(PTH)KIT-EZ -> capacitor-wima:C7.5/3
- LED1, LED2: device adafruit:LED5MM -> adafruit:LED3MM
Connections:
- new net ADC1: AN1.3, U$1.PC1
- new net ADC3: AN1.4, U$1.PC3
- new net N$10: AN1.2, JP1.2
- net 3.3V: now also JP1.3
- net 5V: now also JP1.1
- net GND: now also AN1.5, AN1.6
Other:
- moved on the sheet: C2
Changed lines of the file:
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@@
 <part name="LED_PWR" library="adafruit" deviceset="LED" device="5MM"/>
 <part name="IC2" library="SparkFun-PowerIC" deviceset="V_REG_78XX" device="-TO-220"/>
-<part name="C2" library="SparkFun-Capacitors" deviceset="0.1UF-50V-20%(PTH)" device="KIT-EZ"/>
+<part name="C2" library="capacitor-wima" deviceset="C" device="7.5/3"/>
 <part name="C3" library="SparkFun-Capacitors" deviceset="0.1UF-50V-20%(PTH)" device="KIT-EZ"/>
 <part name="GND25" library="SparkFun-Aesthetics" deviceset="GND" device=""/>
@@
 <part name="SUPPLY29" library="SparkFun-Aesthetics" deviceset="5V" device=""/>
 <part name="GND29" library="SparkFun-Aesthetics" deviceset="GND" device=""/>
-<part name="LED1" library="adafruit" deviceset="LED" device="5MM"/>
-<part name="LED2" library="adafruit" deviceset="LED" device="5MM"/>
+<part name="LED1" library="adafruit" deviceset="LED" device="3MM"/>
+<part name="LED2" library="adafruit" deviceset="LED" device="3MM"/>
 <part name="R9" library="adafruit" deviceset="R-US_" device="0204/2V"/>
 <part name="R10" library="adafruit" deviceset="R-US_" device="0204/2V"/>
@@
 <part name="SUPPLY7" library="SparkFun-Aesthetics" deviceset="3.3V" device=""/>
 <part name="R11" library="adafruit" deviceset="R-US_" device="M1406"/>
+<part name="AN1" library="con-tycoelectronics" deviceset="RJ11" device="" technology="-2L-B"/>
+<part name="GND18" library="SparkFun-Aesthetics" deviceset="GND" device=""/>
+<part name="JP1" library="jumper" deviceset="JP2E" device=""/>
+<part name="SUPPLY16" library="SparkFun-Aesthetics" deviceset="3.3V" device=""/>
+<part name="SUPPLY26" library="SparkFun-Aesthetics" deviceset="5V" device=""/>
 </parts>
 <sheets>
@@
 <instance part="SUPPLY7" gate="G$1" x="327.66" y="22.86" rot="MR90"/>
 <instance part="R11" gate="G$1" x="124.46" y="127"/>
+<instance part="AN1" gate="G$1" x="383.54" y="17.78" rot="MR0"/>
+<instance part="GND18" gate="1" x="391.16" y="12.7" rot="R90"/>
+<instance part="JP1" gate="1" x="401.32" y="30.48"/>
+<instance part="SUPPLY16" gate="G$1" x="403.86" y="27.94" rot="MR180"/>
+<instance part="SUPPLY26" gate="G$1" x="398.78" y="27.94" rot="R180"/>
 </instances>
 <busses>
@@
 <pinref part="C2" gate="G$1" pin="2"/>
 <wire x1="330.2" y1="119.38" x2="330.2" y2="121.92" width="0.1524" layer="91"/>
-<wire x1="317.5" y1="121.92" x2="317.5" y2="119.38" width="0.1524" layer="91"/>
 <wire x1="317.5" y1="119.38" x2="330.2" y2="119.38" width="0.1524" layer="91"/>
 <pinref part="C3" gate="G$1" pin="2"/>
@@
 <junction x="287.02" y="76.2"/>
 </segment>
+<segment>
+<pinref part="AN1" gate="G$1" pin="5"/>
+<pinref part="GND18" gate="1" pin="GND"/>
+<wire x1="388.62" y1="12.7" x2="386.08" y2="12.7" width="0.1524" layer="91"/>
+<pinref part="AN1" gate="G$1" pin="6"/>
+<wire x1="386.08" y1="10.16" x2="386.08" y2="12.7" width="0.1524" layer="91"/>
+<junction x="386.08" y="12.7"/>
+</segment>
 </net>
 <net name="5V" class="0">
@@
 <wire x1="287.02" y1="86.36" x2="289.56" y2="86.36" width="0.1524" layer="91"/>
 </segment>
+<segment>
+<pinref part="JP1" gate="1" pin="1"/>
+<pinref part="SUPPLY26" gate="G$1" pin="5V"/>
+</segment>
 </net>
 <net name="3.3V" class="0">
@@
 <pinref part="R11" gate="G$1" pin="1"/>
 <wire x1="116.84" y1="127" x2="119.38" y2="127" width="0.1524" layer="91"/>
+</segment>
+<segment>
+<pinref part="JP1" gate="1" pin="3"/>
+<pinref part="SUPPLY16" gate="G$1" pin="3.3V"/>
 </segment>
 </net>
@@
 <pinref part="IC2" gate="G$1" pin="IN"/>
 <pinref part="C2" gate="G$1" pin="1"/>
-<wire x1="317.5" y1="129.54" x2="322.58" y2="129.54" width="0.1524" layer="91"/>
-<wire x1="317.5" y1="129.54" x2="314.96" y2="129.54" width="0.1524" layer="91"/>
+<wire x1="317.5" y1="127" x2="322.58" y2="129.54" width="0.1524" layer="91"/>
+<wire x1="317.5" y1="127" x2="314.96" y2="129.54" width="0.1524" layer="91"/>
 <pinref part="SUPPLY23" gate="1" pin="VCC"/>
-<junction x="317.5" y="129.54"/>
+<junction x="317.5" y="127"/>
 </segment>
 <segment>
@@
 </segment>
 </net>
+<net name="ADC1" class="0">
+<segment>
+<pinref part="U$1" gate="G$1" pin="PC1"/>
+<wire x1="25.4" y1="60.96" x2="2.54" y2="60.96" width="0.1524" layer="91"/>
+<label x="2.54" y="60.96" size="1.778" layer="95"/>
+</segment>
+<segment>
+<pinref part="AN1" gate="G$1" pin="3"/>
+<wire x1="386.08" y1="17.78" x2="406.4" y2="17.78" width="0.1524" layer="91"/>
+<label x="401.32" y="17.78" size="1.778" layer="95"/>
+</segment>
+</net>
+<net name="ADC3" class="0">
+<segment>
+<pinref part="U$1" gate="G$1" pin="PC3"/>
+<wire x1="25.4" y1="58.42" x2="2.54" y2="58.42" width="0.1524" layer="91"/>
+<label x="2.54" y="58.42" size="1.778" layer="95"/>
+</segment>
+<segment>
+<pinref part="AN1" gate="G$1" pin="4"/>
+<wire x1="386.08" y1="15.24" x2="406.4" y2="15.24" width="0.1524" layer="91"/>
+<label x="401.32" y="15.24" size="1.778" layer="95"/>
+</segment>
+</net>
+<net name="N$10" class="0">
+<segment>
+<pinref part="AN1" gate="G$1" pin="2"/>
+<pinref part="JP1" gate="1" pin="2"/>
+<wire x1="386.08" y1="20.32" x2="401.32" y2="20.32" width="0.1524" layer="91"/>
+<wire x1="401.32" y1="20.32" x2="401.32" y2="27.94" width="0.1524" layer="91"/>
+</segment>
+</net>

Commit message: Realizado o roteamento Dual-Layer para fresamento.
Aumento de espacamento (trilhas de 24mil, espacamento 24mil)
Parts:
- R1, R3: device adafruit:R-US_M1406 -> adafruit:R-US_0204/5
- R10, R9: device adafruit:R-US_0204/2V -> rcl:R-EU_0204/2V
- SJ1: device jumper:SJ2WW -> con-lstb:MA03-1
Connections:
- new net PA7/PWM: LED1.C, U$1.PA7
- new net PE7: RECV.1, U$1.PE7
- net PB0/PWM: no longer LED2.C
- net PB1/PWM: now also LED2.C; no longer LED1.C
- net PB3/SPI1_SCK: now also SPI1.4; no longer SPI1.2
- net PB5/SPI1_MOSI: now also SPI1.2; no longer SPI1.4
- net PE11/PWM: now also SV2.1; no longer SV1.1
- net PE13/PWM: now also SV3.1; no longer SV2.1
- net PE14/PWM: no longer SV3.1
- net PE9/PWM: now also SV1.1; no longer RECV.1

Commit message: Corrigido o conversor logico invertido e a pinagem incorreta de algumas portas.
Connections:
- net 5V: now also I2C1_ESC.1, I2C3_IMU.1, LED1.A, LED2.A; no longer R10.1, R9.1
- net N$1: now also SV4.2; no longer SV4.6
- net N$10: now also AN1.1; no longer AN1.2
- net N$2: now also SV4.1, U$2.B_L; no longer SV4.5, U$2.C_L
- net N$5: now also LED1.C, R9.1; no longer LED1.A, R9.2
- net N$7: now also LED2.C, R10.1; no longer LED2.A, R10.2
- net PA7/PWM: now also R9.2; no longer LED1.C
- net PB1/PWM: now also R10.2; no longer LED2.C
- net PB8/I2C1_SCL: now also U$2.C_L; no longer U$2.B_L
- net SCL1: now also U$2.C_H; no longer U$2.B_H
- net SCL2: now also SV4.5, U$2.B_H; no longer SV4.1, U$2.C_H
- net SDA2: now also SV4.6; no longer SV4.2
Other:
- note added: "R11 apenas para 'pular' uma trilha no esquematico."
- moved on the sheet: JP1, LED1, LED2, R10, R11, R9
