File: electronics/stm32f4discovery-shield/schematic.brd (EAGLE design)
At the start: 135.6 x 110.5 mm, 40 parts, among them IC1 MAX3468CPA, IC3 LM340H-12, IC4 LM340H-12, J1 POWER_JACKSLT, Q1 BC548

Commit message: Iniciando revisao da shield Discovery.
Parts:
- moved I2C1_ESC 5.08 mm to (100.3, 83.2)
- moved ESC 0.64 mm to (85.1, 83.2)
Routing:
- net GND: track 39.6 -> 70.3 mm
- net 5V: track 311.2 -> 320.0 mm
- net SDA1: track 15.3 -> 22.8 mm
- net SCL1: track 18.1 -> 25.6 mm
Changed lines of the file:
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@@
 <?xml version="1.0" encoding="utf-8"?>
 <!DOCTYPE eagle SYSTEM "eagle.dtd">
-<eagle version="6.5.0">
+<eagle version="6.4">
 <drawing>
 <settings>
@@
 <setting verticaltext="up"/>
 </settings>
-<grid distance="0.05" unitdist="inch" unit="inch" style="lines" multiple="1" display="yes" altdistance="0.025" altunitdist="inch" altunit="inch"/>
+<grid distance="0.025" unitdist="inch" unit="inch" style="lines" multiple="1" display="yes" altdistance="0.025" altunitdist="inch" altunit="inch"/>
 <layers>
 <layer number="1" name="Top" color="4" fill="1" visible="yes" active="yes"/>
@@
 <element name="U$1" library="STM32F4-DISCOVERY" package="STM32F4-DISCOVERY" value="STM32F4-DISCOVERY" x="52.07" y="40.64"/>
 <element name="U$2" library="provant_custom" package="JYMCU_LOGIC_LEVEL_SHIFTER_DIP" value="JYMCU_LOGIC_LEVEL_CONVERTER" x="91.44" y="64.135" rot="R90"/>
-<element name="I2C1_ESC" library="con-tycoelectronics" package="RJ11-NO_SHIELD" value="RJ11-2L-B" x="100.33" y="78.105" rot="R90">
-<attribute name="OC_NEWARK" value="83F4463" x="100.33" y="78.105" size="1.778" layer="27" rot="R90" display="off"/>
-<attribute name="MPN" value="RJ11-2L-B" x="100.33" y="78.105" size="1.778" layer="27" rot="R90" display="off"/>
-<attribute name="MF" value="TYCO ELECTRONICS" x="100.33" y="78.105" size="1.778" layer="27" rot="R90" display="off"/>
-<attribute name="OC_FARNELL" value="unknown" x="100.33" y="78.105" size="1.778" layer="27" rot="R90" display="off"/>
+<element name="I2C1_ESC" library="con-tycoelectronics" package="RJ11-NO_SHIELD" value="RJ11-2L-B" x="100.33" y="83.185" rot="R90">
+<attribute name="OC_NEWARK" value="83F4463" x="100.33" y="83.185" size="1.778" layer="27" rot="R90" display="off"/>
+<attribute name="MPN" value="RJ11-2L-B" x="100.33" y="83.185" size="1.778" layer="27" rot="R90" display="off"/>
+<attribute name="MF" value="TYCO ELECTRONICS" x="100.33" y="83.185" size="1.778" layer="27" rot="R90" display="off"/>
+<attribute name="OC_FARNELL" value="unknown" x="100.33" y="83.185" size="1.778" layer="27" rot="R90" display="off"/>
 </element>
 <element name="I2C3_IMU" library="con-tycoelectronics" package="RJ11-NO_SHIELD" value="RJ11-2L-B" x="100.33" y="46.99" rot="R90">
@@
 <attribute name="OC_FARNELL" value="unknown" x="85.09" y="46.99" size="1.778" layer="27" rot="R90" display="off"/>
 </element>
-<element name="ESC" library="con-lstb" package="MA03-2" value="" x="85.09" y="82.55" rot="R90">
-<attribute name="OC_NEWARK" value="unknown" x="85.09" y="82.55" size="1.778" layer="27" rot="R90" display="off"/>
-<attribute name="MPN" value="" x="85.09" y="82.55" size="1.778" layer="27" rot="R90" display="off"/>
-<attribute name="MF" value="" x="85.09" y="82.55" size="1.778" layer="27" rot="R90" display="off"/>
-<attribute name="OC_FARNELL" value="unknown" x="85.09" y="82.55" size="1.778" layer="27" rot="R90" display="off"/>
+<element name="ESC" library="con-lstb" package="MA03-2" value="" x="85.09" y="83.185" rot="R90">
+<attribute name="OC_NEWARK" value="unknown" x="85.09" y="83.185" size="1.778" layer="27" rot="R90" display="off"/>
+<attribute name="MPN" value="" x="85.09" y="83.185" size="1.778" layer="27" rot="R90" display="off"/>
+<attribute name="MF" value="" x="85.09" y="83.185" size="1.778" layer="27" rot="R90" display="off"/>
+<attribute name="OC_FARNELL" value="unknown" x="85.09" y="83.185" size="1.778" layer="27" rot="R90" display="off"/>
 </element>
 <element name="IC1" library="maxim" package="DIL08" value="MAX3468CPA" x="62.5475" y="62.23">
@@
 <contactref element="SPI1" pad="6"/>
 <contactref element="SPI1" pad="5"/>
-<wire x1="6.35" y1="41.275" x2="3.81" y2="35.56" width="0" layer="19" extent="1-1"/>
+<wire x1="87.63" y1="70.485" x2="88.9" y2="71.755" width="0.4064" layer="16"/>
+<wire x1="6.35" y1="41.275" x2="6.35" y2="39.37" width="0.4064" layer="16"/>
+<wire x1="24.13" y1="43.18" x2="25.4" y2="41.91" width="0.4064" layer="16"/>
+<wire x1="25.4" y1="41.91" x2="27.94" y2="41.91" width="0.4064" layer="16"/>
+<wire x1="6.35" y1="39.37" x2="8.255" y2="39.37" width="0.4064" layer="16"/>
+<wire x1="8.255" y1="39.37" x2="10.795" y2="36.83" width="0.4064" layer="16"/>
+<wire x1="10.795" y1="36.83" x2="27.94" y2="36.83" width="0.4064" layer="16"/>
+<wire x1="6.35" y1="39.37" x2="3.81" y2="35.56" width="0" layer="19" extent="16-16"/>
 <wire x1="91.44" y1="15.875" x2="82.55" y2="16.1925" width="0" layer="19" extent="1-1"/>
-<wire x1="87.63" y1="70.485" x2="86.36" y2="80.01" width="0" layer="19" extent="1-1"/>
-<wire x1="24.13" y1="10.16" x2="12.7" y2="12.065" width="0" layer="19" extent="1-1"/>
 <wire x1="27.4955" y1="80.01" x2="26.67" y2="71.12" width="0" layer="19" extent="1-1"/>
 <wire x1="12.7" y1="67.945" x2="24.13" y2="66.04" width="0" layer="19" extent="1-1"/>
 <wire x1="10.16" y1="66.675" x2="12.7" y2="67.945" width="0" layer="19" extent="1-1"/>
-<wire x1="91.44" y1="32.385" x2="93.98" y2="17.145" width="0" layer="19" extent="1-1"/>
-<wire x1="24.13" y1="43.18" x2="6.35" y2="41.275" width="0" layer="19" extent="1-1"/>
+<wire x1="93.98" y1="33.655" x2="91.44" y2="48.895" width="0" layer="19" extent="1-1"/>
 </signal>
 <signal name="5V">
@@
 <wire x1="91.44" y1="27.305" x2="92.71" y2="26.035" width="0.4064" layer="16"/>
 <wire x1="92.71" y1="26.035" x2="96.52" y2="26.035" width="0.4064" layer="16"/>
-<wire x1="96.52" y1="74.295" x2="93.98" y2="76.2" width="0" layer="19" extent="16-16"/>
+<wire x1="96.52" y1="74.295" x2="96.52" y2="80.01" width="0.4064" layer="16"/>
+<wire x1="96.52" y1="80.01" x2="95.25" y2="81.28" width="0.4064" layer="16"/>
+<wire x1="95.25" y1="81.28" x2="93.98" y2="81.28" width="0.4064" layer="16"/>
 </signal>
 <signal name="3.3V">
@@
 <contactref element="I2C1_ESC" pad="3"/>
 <contactref element="U$2" pad="AH"/>
-<wire x1="83.82" y1="82.55" x2="86.36" y2="82.55" width="0.4064" layer="16"/>
-<wire x1="96.52" y1="80.645" x2="96.52" y2="79.375" width="0.4064" layer="16"/>
-<wire x1="96.52" y1="79.375" x2="90.17" y2="73.025" width="0.4064" layer="16"/>
-<wire x1="90.17" y1="73.025" x2="90.17" y2="70.485" width="0.4064" layer="16"/>
-<wire x1="90.17" y1="73.025" x2="91.44" y2="77.47" width="0" layer="19" extent="16-16"/>
-<wire x1="86.36" y1="82.55" x2="91.44" y2="77.47" width="0" layer="19" extent="1-1"/>
+<wire x1="83.82" y1="83.185" x2="86.36" y2="83.185" width="0.4064" layer="16"/>
+<wire x1="90.17" y1="70.485" x2="90.17" y2="71.12" width="0.4064" layer="16"/>
+<wire x1="90.17" y1="71.12" x2="91.44" y2="72.39" width="0.4064" layer="16"/>
+<wire x1="91.44" y1="72.39" x2="91.44" y2="77.47" width="0.4064" layer="16"/>
+<wire x1="91.44" y1="77.47" x2="89.535" y2="79.375" width="0.4064" layer="16"/>
+<wire x1="89.535" y1="79.375" x2="89.535" y2="81.915" width="0.4064" layer="16"/>
+<wire x1="89.535" y1="81.915" x2="90.17" y2="82.55" width="0.4064" layer="16"/>
+<wire x1="90.17" y1="82.55" x2="91.44" y2="82.55" width="0.4064" layer="16"/>
+<wire x1="91.44" y1="82.55" x2="88.9" y2="82.55" width="0.4064" layer="16"/>
+<wire x1="88.9" y1="82.55" x2="88.265" y2="83.185" width="0.4064" layer="16"/>
+<wire x1="88.265" y1="83.185" x2="86.36" y2="83.185" width="0.4064" layer="16"/>
 </signal>
 <signal name="SCL1">
@@
 <contactref element="I2C1_ESC" pad="4"/>
 <contactref element="U$2" pad="BH"/>
-<wire x1="88.265" y1="83.185" x2="86.36" y2="85.09" width="0.4064" layer="16"/>
-<wire x1="86.36" y1="85.09" x2="83.82" y2="85.09" width="0.4064" layer="16"/>
-<wire x1="97.79" y1="81.28" x2="97.79" y2="78.74" width="0.4064" layer="16"/>
-<wire x1="97.79" y1="78.74" x2="92.71" y2="73.66" width="0.4064" layer="16"/>
-<wire x1="92.71" y1="73.66" x2="92.71" y2="70.485" width="0.4064" layer="16"/>
-<wire x1="97.79" y1="78.74" x2="93.98" y2="78.74" width="0" layer="19" extent="16-16"/>
-<wire x1="88.265" y1="83.185" x2="93.98" y2="78.74" width="0" layer="19" extent="16-16"/>
+<wire x1="86.36" y1="85.725" x2="83.82" y2="85.725" width="0.4064" layer="16"/>
+<wire x1="92.71" y1="70.485" x2="92.71" y2="83.185" width="0.4064" layer="16"/>
+<wire x1="92.71" y1="83.185" x2="93.345" y2="83.82" width="0.4064" layer="16"/>
+<wire x1="93.345" y1="83.82" x2="93.98" y2="83.82" width="0.4064" layer="16"/>
+<wire x1="93.98" y1="83.82" x2="88.9" y2="83.82" width="0.4064" layer="16"/>
+<wire x1="88.9" y1="83.82" x2="88.265" y2="84.455" width="0.4064" layer="16"/>
+<wire x1="88.265" y1="84.455" x2="88.265" y2="85.09" width="0.4064" layer="16"/>
+<wire x1="88.265" y1="85.09" x2="87.63" y2="85.725" width="0.4064" layer="16"/>
+<wire x1="87.63" y1="85.725" x2="86.36" y2="85.725" width="0.4064" layer="16"/>
 </signal>
 <signal name="PB9/I2C1_SDA">
