File: electronics/stm32f4discovery-shield/schematic-for-manuf.sch (EAGLE design)
At the start: 43 parts, among them IC1 MAX3468CPA, IC3 LM340H-12, IC4 LM340H-12, J1 POWER_JACKSLT, Q1 BC548

Commit message: Introduzido jumper para servo Dongbu.
Parts:
- added JP2: (no value), jumper:JP2QE
Connections:
- net D+/TX: now also JP2-1.2
- net D-/RX: now also JP2-2.2
- net PB6/USART1_TX: now also JP2-1.1
- net PB7/USART1_RX: now also JP2-2.1
Other:
- note added: "* Para os servos RX24f, montar IC1. * Para servos Dongbu, remover IC1, e bypassar linhas de TX e RX atraves de JP2-1 e JP2-2."
- note removed: "* Para os servos RX24f, montar IC1. * Para servos Dongbu, remover IC1, e bypassar linhas de TX e RX atraves de JP1 e JP2."
Changed lines of the file:
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@@
 <?xml version="1.0" encoding="utf-8"?>
 <!DOCTYPE eagle SYSTEM "eagle.dtd">
-<eagle version="6.4">
+<eagle version="6.5.0">
 <drawing>
 <settings>
@@
 <part name="SUPPLY16" library="SparkFun-Aesthetics" deviceset="3.3V" device=""/>
 <part name="SUPPLY26" library="SparkFun-Aesthetics" deviceset="5V" device=""/>
+<part name="JP2" library="jumper" deviceset="JP2QE" device=""/>
 </parts>
 <sheets>
@@
 * IC3 e IC4 nao vem montados por default.</text>
 <text x="175.26" y="167.64" size="1.778" layer="91">* Para os servos RX24f, montar IC1.
-* Para servos Dongbu, remover IC1, e bypassar linhas de TX e RX atraves de JP1 e JP2.</text>
+* Para servos Dongbu, remover IC1, e bypassar linhas de TX e RX atraves de JP2-1 e JP2-2.</text>
 <text x="185.42" y="5.08" size="1.778" layer="91">* Para sonar XL-MaxSonar-EZ MB1200, soldar SJ1 na posiçao 2-3.
 * Para usar como linha de serial comum, soldar SJ1 na posiçao 1-2. </text>
@@
 <instance part="SUPPLY16" gate="G$1" x="406.4" y="35.56" rot="MR180"/>
 <instance part="SUPPLY26" gate="G$1" x="401.32" y="35.56" rot="R180"/>
+<instance part="JP2" gate="-1" x="177.8" y="137.16"/>
+<instance part="JP2" gate="-2" x="185.42" y="137.16"/>
 </instances>
 <busses>
@@
 <label x="271.78" y="119.38" size="1.778" layer="95"/>
 </segment>
+<segment>
+<pinref part="JP2" gate="-1" pin="2"/>
+<wire x1="180.34" y1="134.62" x2="180.34" y2="114.3" width="0.1524" layer="91"/>
+<label x="180.34" y="114.3" size="1.778" layer="95" rot="R90"/>
+</segment>
 </net>
 <net name="D-/RX" class="0">
@@
 <label x="271.78" y="121.92" size="1.778" layer="95"/>
 </segment>
+<segment>
+<pinref part="JP2" gate="-2" pin="2"/>
+<wire x1="187.96" y1="134.62" x2="187.96" y2="114.3" width="0.1524" layer="91"/>
+<label x="187.96" y="114.3" size="1.778" layer="95" rot="R90"/>
+</segment>
 </net>
 <net name="PB6/USART1_TX" class="0">
@@
 <label x="88.9" y="40.64" size="1.778" layer="95"/>
 </segment>
+<segment>
+<pinref part="JP2" gate="-1" pin="1"/>
+<wire x1="177.8" y1="134.62" x2="177.8" y2="114.3" width="0.1524" layer="91"/>
+<label x="177.8" y="114.3" size="1.778" layer="95" rot="R90"/>
+</segment>
 </net>
 <net name="PB7/USART1_RX" class="0">
@@
 <label x="147.32" y="40.64" size="1.778" layer="95"/>
 </segment>
-</net>
+<segment>
+<pinref part="JP2" gate="-2" pin="1"/>
+<wire x1="185.42" y1="134.62" x2="185.42" y2="114.3" width="0.1524" layer="91"/>
+<label x="185.42" y="114.3" size="1.778" layer="95" rot="R90"/>
+</segment>
+</net>
